File: Hardware/Low_Current_Driver/Battery_Management.kicad_sch (KiCad schematic)
At the start: 49 parts, among them J4 Conn_02x07_Odd_Even, Q1 Si4447ADY, Q2 IRF8707PbF, SW1 DPDT_Hirose, U1 LM4040DBZ-5, U2 LM4040DBZ-5, U3 LM393

Commit message: Replicate coil drive channel via native multichannel sheets
Root schematic now instantiates Channel_Outputs.kicad_sch twice as
Coil_Drive_A / Coil_Drive_B, with DAC_OPA.kicad_sch added as a sub-sheet
of DAC.kicad_sch (also instantiated twice). PCB relaid out to match.

Also drops the abandoned ESP32-S3 leftovers (footprint file and the
sym-lib-table entry pointing at an absolute path), removes the stale
Low_Current_Driver-cache legacy lib entry, and adds the STEP models
referenced by the board under 3DModels/.

Co-Authored-By: Claude Opus 4.8 <noreply@anthropic.com>
Other:
- company: Strathclyde University -> QUBIC MEG Lab
- title: "Vernier" Low Current Driver - LCD -> FieldZero Coil Driver - Low Current Driver (2 ch, +/-10 mA)
Changed lines of the file:
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@@
 	(paper "A4")
 	(title_block
-		(title "\"Vernier\" Low Current Driver - LCD")
-		(date "2021-05-18")
-		(rev "1.1.0")
-		(company "Strathclyde University")
-		(comment 1 "Designed by: Marcin Mrozowski")
-		(comment 2 "Checked by: ")
+		(title "FieldZero Coil Driver - Low Current Driver (2 ch, +/-10 mA)")
+		(date "2026-07-22")
+		(rev "0.1")
+		(company "QUBIC MEG Lab")
+		(comment 1 "Designed by: Kayzer")
+		(comment 2 "Checked by:")
 		(comment 3 "Approved by:")
+		(comment 4 "Derived from the Vernier Current Driver - M. Mrozowski, Strathclyde EQOP (arXiv:2207.10348)")
 	)
 	(text "PG LEDs"
