File: Hardware/Low_Current_Driver/MCU.kicad_sch (KiCad schematic)
At the start: 8 parts

Commit message: Replicate coil drive channel via native multichannel sheets
Root schematic now instantiates Channel_Outputs.kicad_sch twice as
Coil_Drive_A / Coil_Drive_B, with DAC_OPA.kicad_sch added as a sub-sheet
of DAC.kicad_sch (also instantiated twice). PCB relaid out to match.

Also drops the abandoned ESP32-S3 leftovers (footprint file and the
sym-lib-table entry pointing at an absolute path), removes the stale
Low_Current_Driver-cache legacy lib entry, and adds the STEP models
referenced by the board under 3DModels/.

Co-Authored-By: Claude Opus 4.8 <noreply@anthropic.com>
Parts:
- removed TP23, TP24, TP25, TP26, TP27: TestPoint_Probe, TestPoint:TestPoint_Pad_D1.0mm, symbol Connector:TestPoint_Probe
- A1: value Arduino_Nano_Every -> Arduino_Nano_R4; DigiKey https://www.digikey.com/en/products/detail/arduino/ABX00028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 -> https://www.digikey.com/en/products/detail/arduino/ABX00143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; MPN ABX00028 -> ABX00143
Connections:
- net GNDD renamed GND
Other:
- note removed: "diode to stop backpowering 9V rail when powering nano with USB"
- company: Strathclyde University -> QUBIC MEG Lab
- title: "Vernier" Low Current Driver - LCD -> FieldZero Coil Driver - Low Current Driver (2 ch, +/-10 mA)
