File: Hardware/Low_Current_Driver/Mounting_Holes.kicad_sch (KiCad schematic)
At the start: 5 parts

Commit message: Replicate coil drive channel via native multichannel sheets
Root schematic now instantiates Channel_Outputs.kicad_sch twice as
Coil_Drive_A / Coil_Drive_B, with DAC_OPA.kicad_sch added as a sub-sheet
of DAC.kicad_sch (also instantiated twice). PCB relaid out to match.

Also drops the abandoned ESP32-S3 leftovers (footprint file and the
sym-lib-table entry pointing at an absolute path), removes the stale
Low_Current_Driver-cache legacy lib entry, and adds the STEP models
referenced by the board under 3DModels/.

Co-Authored-By: Claude Opus 4.8 <noreply@anthropic.com>
Parts:
- H1: footprint MountingHole:MountingHole_3.2mm_M3_Pad_Via -> MountingHole:MountingHole_2.2mm_M2_DIN965_Pad
Connections:
- net GNDA renamed GND
Other:
- company: Strathclyde University -> QUBIC MEG Lab
- title: "Vernier" Low Current Driver - LCD -> FieldZero Coil Driver - Low Current Driver (2 ch, +/-10 mA)
Changed lines of the file:
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@@
 	(paper "A4")
 	(title_block
-		(title "\"Vernier\" Low Current Driver - LCD")
-		(date "2021-05-18")
-		(rev "1.1.0")
-		(company "Strathclyde University")
-		(comment 1 "Designed by: Marcin Mrozowski")
-		(comment 2 "Checked by: ")
+		(title "FieldZero Coil Driver - Low Current Driver (2 ch, +/-10 mA)")
+		(date "2026-07-22")
+		(rev "0.1")
+		(company "QUBIC MEG Lab")
+		(comment 1 "Designed by: Kayzer")
+		(comment 2 "Checked by:")
 		(comment 3 "Approved by:")
+		(comment 4 "Derived from the Vernier Current Driver - M. Mrozowski, Strathclyde EQOP (arXiv:2207.10348)")
 	)
 	(symbol
@@
 		)
 		(instances
-			(project "Low_Current_Driver"
-				(path "/f3b999b2-351b-4bd9-b912-3db082ddbf64/00000000-0000-0000-0000-00005eb165a9"
+			(project "Mounting_Holes"
+				(path "/9b211199-dde8-45c5-9f80-9565c0466fbc"
 					(reference "H4")
 					(unit 1)
 				)
 			)
-		)
-	)
-	(symbol
-		(lib_id "power:GNDA")
+			(project "Low_Current_Driver"
+				(path "/f3b999b2-351b-4bd9-b912-3db082ddbf64/00000000-0000-0000-0000-00005eb165a9"
+					(reference "H4")
+					(unit 1)
+				)
+			)
+		)
+	)
+	(symbol
+		(lib_id "power:GND")
 		(at 36.83 111.76 0)
 		(unit 1)
@@
 			)
 		)
-		(property "Value" "GNDA"
+		(property "Value" "GND"
 			(at 36.957 116.1542 0)
 			(show_name no)
@@
 		)
 		(instances
+			(project "Mounting_Holes"
+				(path "/9b211199-dde8-45c5-9f80-9565c0466fbc"
+					(reference "#PWR0206")
+					(unit 1)
+				)
+			)
 			(project "Low_Current_Driver"
 				(path "/f3b999b2-351b-4bd9-b912-3db082ddbf64/00000000-0000-0000-0000-00005eb165a9"
@@
 		)
 		(instances
-			(project "Low_Current_Driver"
-				(path "/f3b999b2-351b-4bd9-b912-3db082ddbf64/00000000-0000-0000-0000-00005eb165a9"
+			(project "Mounting_Holes"
+				(path "/9b211199-dde8-45c5-9f80-9565c0466fbc"
 					(reference "H3")
 					(unit 1)
 				)
 			)
-		)
-	)
-	(symbol
-		(lib_id "power:GNDA")
+			(project "Low_Current_Driver"
+				(path "/f3b999b2-351b-4bd9-b912-3db082ddbf64/00000000-0000-0000-0000-00005eb165a9"
+					(reference "H3")
+					(unit 1)
+				)
+			)
+		)
+	)
+	(symbol
+		(lib_id "power:GND")
 		(at 36.83 99.06 0)
 		(unit 1)
@@
 			)
 		)
-		(property "Value" "GNDA"
+		(property "Value" "GND"
 			(at 36.957 103.4542 0)
 			(show_name no)
@@
 		)
 		(instances
+			(project "Mounting_Holes"
+				(path "/9b211199-dde8-45c5-9f80-9565c0466fbc"
+					(reference "#PWR0207")
+					(unit 1)
+				)
+			)
 			(project "Low_Current_Driver"
 				(path "/f3b999b2-351b-4bd9-b912-3db082ddbf64/00000000-0000-0000-0000-00005eb165a9"
@@
 		)
 		(instances
-			(project "Low_Current_Driver"
-				(path "/f3b999b2-351b-4bd9-b912-3db082ddbf64/00000000-0000-0000-0000-00005eb165a9"
+			(project "Mounting_Holes"
+				(path "/9b211199-dde8-45c5-9f80-9565c0466fbc"
 					(reference "H2")
 					(unit 1)
 				)
 			)
-		)
-	)
-	(symbol
-		(lib_id "power:GNDA")
+			(project "Low_Current_Driver"
+				(path "/f3b999b2-351b-4bd9-b912-3db082ddbf64/00000000-0000-0000-0000-00005eb165a9"
+					(reference "H2")
+					(unit 1)
+				)
+			)
+		)
+	)
+	(symbol
+		(lib_id "power:GND")
 		(at 36.83 87.63 0)
 		(unit 1)
@@
 			)
 		)
-		(property "Value" "GNDA"
+		(property "Value" "GND"
 			(at 36.957 92.0242 0)
 			(show_name no)
@@
 		)
 		(instances
+			(project "Mounting_Holes"
+				(path "/9b211199-dde8-45c5-9f80-9565c0466fbc"
+					(reference "#PWR0208")
+					(unit 1)
+				)
+			)
 			(project "Low_Current_Driver"
 				(path "/f3b999b2-351b-4bd9-b912-3db082ddbf64/00000000-0000-0000-0000-00005eb165a9"
@@
 			)
 		)
-		(property "Footprint" "MountingHole:MountingHole_3.2mm_M3_Pad_Via"
+		(property "Footprint" "MountingHole:MountingHole_2.2mm_M2_DIN965_Pad"
 			(at 36.83 73.66 0)
 			(hide yes)
@@
 		)
 		(instances
-			(project "Low_Current_Driver"
-				(path "/f3b999b2-351b-4bd9-b912-3db082ddbf64/00000000-0000-0000-0000-00005eb165a9"
+			(project "Mounting_Holes"
+				(path "/9b211199-dde8-45c5-9f80-9565c0466fbc"
 					(reference "H1")
 					(unit 1)
 				)
 			)
-		)
-	)
-	(symbol
-		(lib_id "power:GNDA")
+			(project "Low_Current_Driver"
+				(path "/f3b999b2-351b-4bd9-b912-3db082ddbf64/00000000-0000-0000-0000-00005eb165a9"
+					(reference "H1")
+					(unit 1)
+				)
+			)
+		)
+	)
+	(symbol
+		(lib_id "power:GND")
 		(at 36.83 76.2 0)
 		(unit 1)
@@
 			)
 		)
-		(property "Value" "GNDA"
+		(property "Value" "GND"
 			(at 36.957 80.5942 0)
 			(show_name no)
@@
 		)
 		(instances
+			(project "Mounting_Holes"
+				(path "/9b211199-dde8-45c5-9f80-9565c0466fbc"
+					(reference "#PWR0209")
+					(unit 1)
+				)
+			)
 			(project "Low_Current_Driver"
 				(path "/f3b999b2-351b-4bd9-b912-3db082ddbf64/00000000-0000-0000-0000-00005eb165a9"
@@
 		)
 		(instances
-			(project "Low_Current_Driver"
-				(path "/f3b999b2-351b-4bd9-b912-3db082ddbf64/00000000-0000-0000-0000-00005eb165a9"
+			(project "Mounting_Holes"
+				(path "/9b211199-dde8-45c5-9f80-9565c0466fbc"
 					(reference "H5")
 					(unit 1)
 				)
 			)
-		)
-	)
-	(symbol
-		(lib_id "power:GNDA")
+			(project "Low_Current_Driver"
+				(path "/f3b999b2-351b-4bd9-b912-3db082ddbf64/00000000-0000-0000-0000-00005eb165a9"
+					(reference "H5")
+					(unit 1)
+				)
+			)
+		)
+	)
+	(symbol
+		(lib_id "power:GND")
 		(at 58.42 111.76 0)
 		(unit 1)
@@
 			)
 		)
-		(property "Value" "GNDA"
+		(property "Value" "GND"
 			(at 58.547 116.1542 0)
 			(show_name no)
@@
 		)
 		(instances
-			(project "Low_Current_Driver"
-				(path "/f3b999b2-351b-4bd9-b912-3db082ddbf64/00000000-0000-0000-0000-00005eb165a9"
+			(project "Mounting_Holes"
+				(path "/9b211199-dde8-45c5-9f80-9565c0466fbc"
 					(reference "#PWR0210")
 					(unit 1)
 				)
 			)
-		)
-	)
+			(project "Low_Current_Driver"
+				(path "/f3b999b2-351b-4bd9-b912-3db082ddbf64/00000000-0000-0000-0000-00005eb165a9"
+					(reference "#PWR0210")
+					(unit 1)
+				)
+			)
+		)
+	)
+	(sheet_instances
+		(path "/"
+			(page "1")
+		)
+	)
+	(embedded_fonts no)
 )
