File: Hardware/Low_Current_Driver/Channel_Outputs.kicad_sch (KiCad schematic)
At the start: 30 parts, among them U12 OPA2210, U13 OPA2210

Commit message: Checkpoint before channel-replication refactor
Snapshot of schematic/PCB work-in-progress prior to restructuring
Channel_Outputs into a reusable hierarchical channel sheet for
replicate-layout. Adds DPST relay footprint.

Co-Authored-By: Claude Opus 4.8 <noreply@anthropic.com>
Connections:
- net U12Bout: now reaches C54.1, R44.1, R45.1, U12.7
- net U12Bin-: now reaches C54.2, R38.1, R44.2, U12.6 (-)
- net U13Bout: now reaches C55.1, R46.1, R47.1, U13.7
- net U13Bin-: now reaches C55.2, R40.1, R46.2, U13.6 (-)
Changed lines of the file:
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@@
+		)
+	)
+	(label "U13Bin+"
+		(at 156.21 102.87 180)
+		(effects
+			(font
+				(size 1.27 1.27)
+			)
+			(justify right bottom)
+		)
+	)
+	(label "U12Bin+"
+		(at 156.21 41.91 180)
+		(effects
+			(font
+				(size 1.27 1.27)
+			)
+			(justify right bottom)
+		)
+	)
+	(label "U12Bout"
+		(at 171.45 39.37 0)
+		(effects
+			(font
+				(size 1.27 1.27)
+			)
+			(justify left bottom)
+		)
+	)
+	(label "U13Bin-"
+		(at 156.21 97.79 180)
+		(effects
+			(font
+				(size 1.27 1.27)
+			)
+			(justify right bottom)
+		)
+	)
+	(label "U12Bin-"
+		(at 156.21 36.83 180)
+		(effects
+			(font
+				(size 1.27 1.27)
+			)
+			(justify right bottom)
+		)
+	)
+	(label "U13Bout"
+		(at 171.45 100.33 0)
+		(effects
+			(font
+				(size 1.27 1.27)
+			)
+			(justify left bottom)
 		)
 	)

Commit message: Replicate coil drive channel via native multichannel sheets
Root schematic now instantiates Channel_Outputs.kicad_sch twice as
Coil_Drive_A / Coil_Drive_B, with DAC_OPA.kicad_sch added as a sub-sheet
of DAC.kicad_sch (also instantiated twice). PCB relaid out to match.

Also drops the abandoned ESP32-S3 leftovers (footprint file and the
sym-lib-table entry pointing at an absolute path), removes the stale
Low_Current_Driver-cache legacy lib entry, and adds the STEP models
referenced by the board under 3DModels/.

Co-Authored-By: Claude Opus 4.8 <noreply@anthropic.com>
Parts:
- removed C39, C40: 100n, Capacitor_SMD:C_0603_1608Metric_Pad1.08x0.95mm_HandSolder, symbol Device:C_Small
- removed C50, C53: 1u, Capacitor_SMD:C_0603_1608Metric_Pad1.08x0.95mm_HandSolder, symbol Device:C_Small
- removed C55: 4.7u, Capacitor_SMD:C_0603_1608Metric_Pad1.08x0.95mm_HandSolder, symbol Device:C_Small
- removed R33, R36, R40, R46, R47: 1k, Resistor_SMD:R_0603_1608Metric_Pad0.98x0.95mm_HandSolder, symbol Device:R_Small
- removed R41: 249, Resistor_SMD:R_0603_1608Metric_Pad0.98x0.95mm_HandSolder, symbol Device:R_Small
- removed TP32, TP34, TP35, TP36: TestPoint_Probe, TestPoint:TestPoint_Pad_D1.0mm, symbol Connector:TestPoint_Probe
- removed U13: OPA2210, Package_SO:SOIC-8_3.9x4.9mm_P1.27mm, symbol vernier_current_driver:OPA2210
- R38, R44, R45: value 1k -> 249; DigiKey https://www.digikey.com/en/products/detail/yageo/RC0603FR-0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 -> https://www.digikey.com/en/products/detail/susumu/RG1608P-2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; MPN RC0603FR-071KL -> RG1608P-2490-B-T5
- R39: DigiKey https://www.digikey.com/en/products/detail/yageo/RC0603FR-0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 -> https://www.digikey.com/en/products/detail/susumu/RG1608P-2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; MPN RC0603FR-07249RL -> RG1608P-2490-B-T5
Connections:
- net +7V5 renamed +9V
- net -7V5 renamed -9V
- net 4Q_DAC_OUT_1 renamed Vout_dac
- net Coil_Iout_1 renamed Iin_coil
- net GNDA renamed GND
- net U12Bin- renamed HCP_FB
- net U12Bout renamed HCP_Out
Other:
- note added: "Howland bridge: R39*R44 = R45*R38 must hold. All four = 249R 0.1% 25ppm thin film (matched set). Gm = 1/R39 -> +/-10.04 mA at +/-2.5 V full scale. C54 across R44: 249R x 4.7uF = 136 Hz comp. corner."
- note removed: "changed howland resistor to 250 from 1k to increase current to 10mA. To maintain cutoff cap is quadrupled to 4u"
- company: Strathclyde University -> QUBIC MEG Lab
- title: "Vernier" Low Current Driver - LCD -> FieldZero Coil Driver - Low Current Driver (2 ch, +/-10 mA)
- moved on the sheet: C37, C38, C49, C52, C54, R32, R35, R38, R39, R44, R45, TP31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

Commit message: Add fab1 package and update docs to as-built for first prototype
- Add fab1.zip + gerbers/drills (4-layer, 127.75x53mm) for JLC bare-board order
- Rewrite context.md PCB section to as-built: external raw ±9V via J3→SW1,
  no on-board LDOs/battery-mgmt; record removed Power/Battery_Management/
  Mounting_Holes sheets and honest ERC state (2 residual errors on DAC8814
  unused C/D outputs, benign)
- Add "Fabrication — first prototype" section: board stack, $25 JLC NRE fee,
  DRC clean, DigiKey BOM verified Active 2026-07-23
- Finalize channel-replication refactor edits (DAC/DAC_OPA/Channel_Outputs)
- Remove stale DRC violations report

Co-Authored-By: Claude Opus 4.8 <noreply@anthropic.com>
Parts:
- C37, C38: DigiKey https://www.digikey.com/en/products/detail/samsung-electro-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 -> https://www.digikey.com/en/products/detail/kemet/C0603C104K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; MPN CL10B104KB8NNNC -> C0603C104K5RACTU
Changed lines of the file:
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@@
 			)
 		)
-		(property "MPN" "CL10B104KB8NNNC"
+		(property "MPN" "C0603C104K5RACTU"
 			(at 71.12 105.41 0)
 			(hide yes)
@@
 			)
 		)
-		(property "DigiKey" "https://www.digikey.com/en/products/detail/samsung-electro-mechanics/CL10B104KB8NNNC/3886658"
+		(property "DigiKey" "https://www.digikey.com/en/products/detail/kemet/C0603C104K5RACTU/1465594"
 			(at 71.12 105.41 0)
 			(hide yes)
@@
 			)
 		)
-		(property "MPN" "CL10B104KB8NNNC"
+		(property "MPN" "C0603C104K5RACTU"
 			(at 69.85 128.27 0)
 			(hide yes)
@@
 			)
 		)
-		(property "DigiKey" "https://www.digikey.com/en/products/detail/samsung-electro-mechanics/CL10B104KB8NNNC/3886658"
+		(property "DigiKey" "https://www.digikey.com/en/products/detail/kemet/C0603C104K5RACTU/1465594"
 			(at 69.85 128.27 0)
 			(hide yes)
