File: Hardware/Low_Current_Driver/DAC.kicad_sch (KiCad schematic)
At the start: 41 parts, among them U10 OPA2210, U7 LTC6655-2.5, U8 DAC8814, U9 OPA2210

Commit message: Checkpoint before channel-replication refactor
Snapshot of schematic/PCB work-in-progress prior to restructuring
Channel_Outputs into a reusable hierarchical channel sheet for
replicate-layout. Adds DPST relay footprint.

Co-Authored-By: Claude Opus 4.8 <noreply@anthropic.com>
Connections:
- net Vout_B_DAC: now reaches R24.1, R25.1, U10.1, U8.11 (Rfb_B)
- net Iout_B: now reaches U10.2 (-), U8.13 (Iout_B)
- net I_outA: now reaches U8.2 (Iout_A), U9.2 (-)
- net Vout_A_DAC: now reaches R21.1, R22.1, U8.4 (Rfb_A), U9.1
Changed lines of the file:
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@@
+		)
+	)
+	(label "Iout_B"
+		(at 179.07 82.55 0)
+		(effects
+			(font
+				(size 1.27 1.27)
+			)
+			(justify left bottom)
 		)
 	)
@@
 		)
 	)
+	(label "Vout_B_DAC"
+		(at 205.74 85.09 0)
+		(effects
+			(font
+				(size 1.27 1.27)
+			)
+			(justify left bottom)
+		)
+	)
 	(label "Vref_2.5V"
 		(at 215.9 74.93 180)
@@
 		(effects
 			(font
+				(size 1.27 1.27)
+			)
+			(justify left bottom)
+		)
+	)
+	(label "I_outA"
+		(at 177.8 46.99 0)
+		(effects
+			(font
+				(size 1.27 1.27)
+			)
+			(justify left bottom)
+		)
+	)
+	(label "Vout_A_DAC"
+		(at 208.28 49.53 0)
+		(effects
+			(font
+				(size 1.27 1.27)
+			)
+			(justify left bottom)
+		)
+	)
+	(label "Vout_B"
+		(at 256.54 87.63 0)
+		(effects
+			(font
+				(size 1.27 1.27)
+			)
+			(justify left bottom)
+		)
+	)
+	(label "Vout_A"
+		(at 256.54 52.07 0)
+		(effects
+			(font

Commit message: Replicate coil drive channel via native multichannel sheets
Root schematic now instantiates Channel_Outputs.kicad_sch twice as
Coil_Drive_A / Coil_Drive_B, with DAC_OPA.kicad_sch added as a sub-sheet
of DAC.kicad_sch (also instantiated twice). PCB relaid out to match.

Also drops the abandoned ESP32-S3 leftovers (footprint file and the
sym-lib-table entry pointing at an absolute path), removes the stale
Low_Current_Driver-cache legacy lib entry, and adds the STEP models
referenced by the board under 3DModels/.

Co-Authored-By: Claude Opus 4.8 <noreply@anthropic.com>
Parts:
- removed C15, C16, C17, C18, C34, C35: 100n, Capacitor_SMD:C_0603_1608Metric_Pad1.08x0.95mm_HandSolder, symbol Device:C_Small
- removed C21, C22, C24, C25: 1u, Capacitor_SMD:C_0603_1608Metric_Pad1.08x0.95mm_HandSolder, symbol Device:C_Small
- removed C23: 47u, Capacitor_SMD:C_1210_3225Metric_Pad1.33x2.70mm_HandSolder, symbol Device:C_Small
- removed R20, R21, R22, R23, R24, R25, R29, R30: 10k, Resistor_SMD:R_0603_1608Metric_Pad0.98x0.95mm_HandSolder, symbol Device:R_Small
- removed TP17, TP18, TP19, TP20, TP21, TP41, TP42, TP43, TP44, TP47: TestPoint_Probe, TestPoint:TestPoint_Pad_D1.0mm, symbol Connector:TestPoint_Probe
- removed U10, U9: OPA2210, Package_SO:SOIC-8_3.9x4.9mm_P1.27mm, symbol vernier_current_driver:OPA2210
Connections:
- net +5V is gone; now on net +5VD: C29.1, C30.1, U8.7 (VDD)
- net +7V5 is gone; now on net +5VD: C14.1, U7.1 (~{SHDN}), U7.2 (Vin)
- net GND: now also U8.16 (Iout_C), U8.17 (VREF_C), U8.18 (Rfb_C), U8.25 (Rfb_D), U8.26 (VREF_D), U8.27 (Iout_D)
- net Vref_2.5V: now also U7.6 (Vout_S); no longer U8.17 (VREF_C), U8.26 (VREF_D)
- net I_outA renamed DAC_Buffer_A/Iin
- net Iout_B renamed DAC_Buffer_B/Iin
- net Vout_A_DAC renamed DAC_Buffer_A/Rfb
- net Vout_B_DAC renamed DAC_Buffer_B/Rfb
- no-connect marks 4 -> 0
Other:
- added sheet DAC_Buffer_A (DAC_OPA.kicad_sch)
- added sheet DAC_Buffer_B (DAC_OPA.kicad_sch)
- note removed: "4Q DAC"
- note removed: "Four quadrant stage (enables bidirectional current flow) compensated to 160 Hz for lower noise"
- note removed: "OP-AMP decoupling"
- note removed: "Resistors have to match expected impedance of DAC output (balance between noise and power)"
- note removed: "Transimpedance amplifier"
- note removed: "Vref at the amplifiers"
- company: Strathclyde University -> QUBIC MEG Lab
- title: "Vernier" Low Current Driver - LCD -> FieldZero Coil Driver - Low Current Driver (2 ch, +/-10 mA)

Commit message: Add fab1 package and update docs to as-built for first prototype
- Add fab1.zip + gerbers/drills (4-layer, 127.75x53mm) for JLC bare-board order
- Rewrite context.md PCB section to as-built: external raw ±9V via J3→SW1,
  no on-board LDOs/battery-mgmt; record removed Power/Battery_Management/
  Mounting_Holes sheets and honest ERC state (2 residual errors on DAC8814
  unused C/D outputs, benign)
- Add "Fabrication — first prototype" section: board stack, $25 JLC NRE fee,
  DRC clean, DigiKey BOM verified Active 2026-07-23
- Finalize channel-replication refactor edits (DAC/DAC_OPA/Channel_Outputs)
- Remove stale DRC violations report

Co-Authored-By: Claude Opus 4.8 <noreply@anthropic.com>
Parts:
- C14, C30: DigiKey https://www.digikey.com/en/products/detail/samsung-electro-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 -> https://www.digikey.com/en/products/detail/kemet/C0603C104K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; MPN CL10B104KB8NNNC -> C0603C104K5RACTU
Changed lines of the file:
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@@
 			)
 		)
-		(property "MPN" "CL10B104KB8NNNC"
+		(property "MPN" "C0603C104K5RACTU"
 			(at 19.05 38.1 0)
 			(hide yes)
@@
 			)
 		)
-		(property "DigiKey" "https://www.digikey.com/en/products/detail/samsung-electro-mechanics/CL10B104KB8NNNC/3886658"
+		(property "DigiKey" "https://www.digikey.com/en/products/detail/kemet/C0603C104K5RACTU/1465594"
 			(at 19.05 38.1 0)
 			(hide yes)
@@
 			)
 		)
-		(property "MPN" "CL10B104KB8NNNC"
+		(property "MPN" "C0603C104K5RACTU"
 			(at 100.33 181.61 0)
 			(hide yes)
@@
 			)
 		)
-		(property "DigiKey" "https://www.digikey.com/en/products/detail/samsung-electro-mechanics/CL10B104KB8NNNC/3886658"
+		(property "DigiKey" "https://www.digikey.com/en/products/detail/kemet/C0603C104K5RACTU/1465594"
 			(at 100.33 181.61 0)
 			(hide yes)
