File: Hardware/Low_Current_Driver/DAC_OPA.kicad_sch (KiCad schematic)
At the start: 12 parts, among them U11 OPA2210

Commit message: Add fab1 package and update docs to as-built for first prototype
- Add fab1.zip + gerbers/drills (4-layer, 127.75x53mm) for JLC bare-board order
- Rewrite context.md PCB section to as-built: external raw ±9V via J3→SW1,
  no on-board LDOs/battery-mgmt; record removed Power/Battery_Management/
  Mounting_Holes sheets and honest ERC state (2 residual errors on DAC8814
  unused C/D outputs, benign)
- Add "Fabrication — first prototype" section: board stack, $25 JLC NRE fee,
  DRC clean, DigiKey BOM verified Active 2026-07-23
- Finalize channel-replication refactor edits (DAC/DAC_OPA/Channel_Outputs)
- Remove stale DRC violations report

Co-Authored-By: Claude Opus 4.8 <noreply@anthropic.com>
Parts:
- C19, C20, C36: DigiKey https://www.digikey.com/en/products/detail/samsung-electro-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 -> https://www.digikey.com/en/products/detail/kemet/C0603C104K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; MPN CL10B104KB8NNNC -> C0603C104K5RACTU
Changed lines of the file:
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@@
 			)
 		)
-		(property "MPN" "CL10B104KB8NNNC"
+		(property "MPN" "C0603C104K5RACTU"
 			(at 46.99 152.4 0)
 			(hide yes)
@@
 			)
 		)
-		(property "DigiKey" "https://www.digikey.com/en/products/detail/samsung-electro-mechanics/CL10B104KB8NNNC/3886658"
+		(property "DigiKey" "https://www.digikey.com/en/products/detail/kemet/C0603C104K5RACTU/1465594"
 			(at 46.99 152.4 0)
 			(hide yes)
@@
 			)
 		)
-		(property "MPN" "CL10B104KB8NNNC"
+		(property "MPN" "C0603C104K5RACTU"
 			(at 173.99 76.2 0)
 			(hide yes)
@@
 			)
 		)
-		(property "DigiKey" "https://www.digikey.com/en/products/detail/samsung-electro-mechanics/CL10B104KB8NNNC/3886658"
+		(property "DigiKey" "https://www.digikey.com/en/products/detail/kemet/C0603C104K5RACTU/1465594"
 			(at 173.99 76.2 0)
 			(hide yes)
@@
 			)
 		)
-		(property "MPN" "CL10B104KB8NNNC"
+		(property "MPN" "C0603C104K5RACTU"
 			(at 77.47 151.13 0)
 			(hide yes)
@@
 			)
 		)
-		(property "DigiKey" "https://www.digikey.com/en/products/detail/samsung-electro-mechanics/CL10B104KB8NNNC/3886658"
+		(property "DigiKey" "https://www.digikey.com/en/products/detail/kemet/C0603C104K5RACTU/1465594"
 			(at 77.47 151.13 0)
 			(hide yes)
